File: motor_control.brd (EAGLE design)
At the start: 100 x 80 mm, 13 parts, among them IC1 NE555D

Commit message: small improve
Parts:
- moved D2 6.71 mm to (39.1, 31.3), turned to 90 degrees
- moved D1 1.41 mm to (37.9, 36.6)
Routing:
- net N$5: track 28.1 -> 29.4 mm
- net N$9: track 13.4 -> 14.4 mm
- net N$3: track 68.1 -> 67.3 mm
Changed lines of the file:
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@@
 <element name="C1" library="rcl" package="C0805" value="2.7nF" x="33.6" y="23.3" rot="R180"/>
 <element name="C2" library="rcl" package="C0805" value="1nF" x="33.4" y="20.6" rot="R90"/>
-<element name="D1" library="diode" package="SMB" value="" x="38.1" y="35.2" rot="R180"/>
-<element name="D2" library="diode" package="SMB" value="" x="39.4" y="24.6" rot="R180"/>
+<element name="D1" library="diode" package="SMB" value="" x="37.9" y="36.6" rot="R180"/>
+<element name="D2" library="diode" package="SMB" value="" x="39.1" y="31.3" rot="R90"/>
 <element name="R1" library="pot" package="CA6V" value="100k" x="31.1" y="38.6" rot="R270"/>
 <element name="R2" library="rcl" package="R0805" value="100" x="22.7" y="27.8" rot="R90"/>
@@
 <contactref element="R1" pad="E"/>
 <contactref element="D1" pad="C"/>
-<wire x1="30.2" y1="19.565" x2="28.665" y2="19.565" width="0.4064" layer="1"/>
-<wire x1="28.665" y1="19.565" x2="28.3" y2="19.2" width="0.4064" layer="1"/>
-<wire x1="28.3" y1="19.2" x2="28.3" y2="17.6" width="0.4064" layer="1"/>
-<wire x1="28.3" y1="17.6" x2="28.8" y2="17.1" width="0.4064" layer="1"/>
-<wire x1="28.8" y1="17.1" x2="34.1" y2="17.1" width="0.4064" layer="1"/>
-<wire x1="34.1" y1="17.1" x2="41.6" y2="24.6" width="0.4064" layer="1"/>
 <wire x1="28.56" y1="36.06" x2="28.56" y2="37.16" width="0.4064" layer="1"/>
 <wire x1="28.56" y1="37.16" x2="32.4" y2="41" width="0.4064" layer="1"/>
 <wire x1="32.4" y1="41" x2="36.3" y2="41" width="0.4064" layer="1"/>
 <wire x1="36.3" y1="41" x2="40.3" y2="37" width="0.4064" layer="1"/>
-<wire x1="40.3" y1="35.2" x2="40.3" y2="37" width="0.4064" layer="1"/>
-<wire x1="40.3" y1="35.2" x2="40.3" y2="25.9" width="0.4064" layer="1"/>
-<wire x1="40.3" y1="25.9" x2="41.6" y2="24.6" width="0.4064" layer="1"/>
+<wire x1="40.1" y1="36.6" x2="40.3" y2="37" width="0.4064" layer="1"/>
 <wire x1="25" y1="20.835" x2="23.765" y2="20.835" width="0.4064" layer="1"/>
 <wire x1="23.765" y1="20.835" x2="23.3" y2="21.3" width="0.4064" layer="1"/>
@@
 <wire x1="24.1" y1="30.8" x2="24.1" y2="23.6" width="0.4064" layer="1"/>
 <wire x1="24.1" y1="23.6" x2="23.3" y2="22.8" width="0.4064" layer="1"/>
+<wire x1="39.1" y1="29.1" x2="39.1" y2="29.7" width="0.4064" layer="1"/>
+<wire x1="39.1" y1="29.7" x2="40.8" y2="31.4" width="0.4064" layer="1"/>
+<wire x1="40.8" y1="31.4" x2="40.8" y2="35.9" width="0.4064" layer="1"/>
+<wire x1="40.8" y1="35.9" x2="40.1" y2="36.6" width="0.4064" layer="1"/>
+<wire x1="30.2" y1="19.565" x2="28.765" y2="19.565" width="0.4064" layer="1"/>
+<wire x1="28.765" y1="19.565" x2="28.2" y2="19" width="0.4064" layer="1"/>
+<wire x1="28.2" y1="19" x2="28.2" y2="17.7" width="0.4064" layer="1"/>
+<wire x1="28.2" y1="17.7" x2="28.7" y2="17.2" width="0.4064" layer="1"/>
+<wire x1="28.7" y1="17.2" x2="33.8" y2="17.2" width="0.4064" layer="1"/>
+<wire x1="33.8" y1="17.2" x2="39.1" y2="22.5" width="0.4064" layer="1"/>
+<wire x1="39.1" y1="22.5" x2="39.1" y2="29.1" width="0.4064" layer="1"/>
 </signal>
 <signal name="N$4">
@@
 <wire x1="31.465" y1="20.835" x2="31.7" y2="20.6" width="0.4064" layer="1"/>
 <wire x1="31.7" y1="20.6" x2="35.4" y2="20.6" width="0.4064" layer="1"/>
-<wire x1="35.4" y1="20.6" x2="37.2" y2="22.4" width="0.4064" layer="1"/>
-<wire x1="37.2" y1="22.4" x2="37.2" y2="24.6" width="0.4064" layer="1"/>
-<wire x1="33.64" y1="38.6" x2="36.6" y2="38.6" width="0.4064" layer="1"/>
-<wire x1="36.6" y1="38.6" x2="38.2" y2="37" width="0.4064" layer="1"/>
-<wire x1="38.2" y1="37" x2="38.2" y2="25.6" width="0.4064" layer="1"/>
-<wire x1="38.2" y1="25.6" x2="37.2" y2="24.6" width="0.4064" layer="1"/>
+<wire x1="33.64" y1="38.6" x2="37.2" y2="38.6" width="0.4064" layer="1"/>
+<wire x1="37.2" y1="38.6" x2="37.9" y2="37.9" width="0.4064" layer="1"/>
+<wire x1="37.9" y1="37.9" x2="37.9" y2="34.7" width="0.4064" layer="1"/>
+<wire x1="37.9" y1="34.7" x2="39.1" y2="33.5" width="0.4064" layer="1"/>
+<wire x1="39.1" y1="33.5" x2="38.7" y2="33.5" width="0.4064" layer="1"/>
+<wire x1="38.7" y1="33.5" x2="37.3" y2="32.1" width="0.4064" layer="1"/>
+<wire x1="37.3" y1="32.1" x2="37.3" y2="22.5" width="0.4064" layer="1"/>
+<wire x1="37.3" y1="22.5" x2="35.4" y2="20.6" width="0.4064" layer="1"/>
 </signal>
 <signal name="N$9">
 <contactref element="C1" pad="1"/>
 <contactref element="D1" pad="A"/>
-<wire x1="35.9" y1="35.2" x2="35.9" y2="33.7" width="0.4064" layer="1"/>
-<wire x1="35.9" y1="33.7" x2="37" y2="32.6" width="0.4064" layer="1"/>
-<wire x1="37" y1="32.6" x2="37" y2="27.5" width="0.4064" layer="1"/>
-<wire x1="37" y1="27.5" x2="34.8" y2="25.3" width="0.4064" layer="1"/>
-<wire x1="34.8" y1="25.3" x2="34.8" y2="23.55" width="0.4064" layer="1"/>
-<wire x1="34.8" y1="23.55" x2="34.55" y2="23.3" width="0.4064" layer="1"/>
+<wire x1="35.7" y1="36.6" x2="35.7" y2="33.7" width="0.4064" layer="1"/>
+<wire x1="35.7" y1="33.7" x2="36.5" y2="32.9" width="0.4064" layer="1"/>
+<wire x1="36.5" y1="32.9" x2="36.5" y2="25.25" width="0.4064" layer="1"/>
+<wire x1="36.5" y1="25.25" x2="34.55" y2="23.3" width="0.4064" layer="1"/>
 </signal>
 <signal name="N$10">

Commit message: some changes
Parts:
- moved C1 1.84 mm to (35.0, 24.5), turned to 225 degrees
- moved C2 1.02 mm to (33.6, 21.6), turned to 135 degrees
- moved IC1 0.58 mm to (27.9, 20.7)
Routing:
- net N$9: track 14.4 -> 11.7 mm
- net N$3: track 67.3 -> 65.5 mm
- net V+: track 34.8 -> 36.3 mm
- net N$5: track 29.4 -> 28.1 mm
- net N$4: track 3.76 -> 4.66 mm

Commit message: added tx signal + led
Parts:
- moved TP2 5.61 mm to (23.4, 38.5)
- moved TP1 3.69 mm to (13.8, 32.5)
- moved IC1 1.66 mm to (27.0, 22.1), turned to 225 degrees
Routing:
- net V+: track 36.3 -> 31.8 mm
- net N$4: track 4.66 -> 8.12 mm
- net N$7: track 9.06 -> 5.75 mm
- net GND: track 18.6 -> 15.4 mm
- net N$5: track 28.1 -> 30.0 mm
