File: laminator.brd (EAGLE design)
At the start: 100 x 80 mm, 9 parts, among them T1 BT138-H

Commit message: laminator board
Parts:
- moved R4 52.1 mm to (39.4, 12.7)
- moved TEN 37.4 mm to (8.89, 10.2)
- moved V220 37.4 mm to (16.5, 10.2)
- moved C1 36.8 mm to (29.2, 6.35)
- moved R2 32.1 mm to (29.2, 8.89), turned to 180 degrees
- moved R3 28.7 mm to (22.9, 6.35), turned to 180 degrees
- moved R1 24.0 mm to (22.9, 8.89), turned to 180 degrees
- moved T1 23.2 mm to (14.0, 26.7)
- moved OK1 7.41 mm to (27.9, 15.2), turned to 90 degrees
Routing:
- net N$4: track 0.00 -> 61.4 mm
- net N$2: track 0.00 -> 24.4 mm
- net N$3: track 0.00 -> 21.4 mm
- net N$7: track 0.00 -> 13.8 mm
- net N$6: track 0.00 -> 3.98 mm
- net N$1: track 0.00 -> 3.87 mm
Changed lines of the file:
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@@
 </autorouter>
 <elements>
-<element name="OK1" library="optocoupler" package="DIL06" value="MOC3041M" x="24.13" y="21.59">
-<attribute name="OC_FARNELL" value="1086677" x="24.13" y="21.59" size="1.778" layer="27" display="off"/>
-<attribute name="OC_NEWARK" value="78K6090" x="24.13" y="21.59" size="1.778" layer="27" display="off"/>
-<attribute name="MF" value="FAIRCHILD SEMICONDUCTOR" x="24.13" y="21.59" size="1.778" layer="27" display="off"/>
-<attribute name="MPN" value="MOC3041M" x="24.13" y="21.59" size="1.778" layer="27" display="off"/>
+<element name="OK1" library="optocoupler" package="DIL06" value="MOC3041M" x="27.94" y="15.24" rot="R90">
+<attribute name="OC_FARNELL" value="1086677" x="27.94" y="15.24" size="1.778" layer="27" rot="R90" display="off"/>
+<attribute name="OC_NEWARK" value="78K6090" x="27.94" y="15.24" size="1.778" layer="27" rot="R90" display="off"/>
+<attribute name="MF" value="FAIRCHILD SEMICONDUCTOR" x="27.94" y="15.24" size="1.778" layer="27" rot="R90" display="off"/>
+<attribute name="MPN" value="MOC3041M" x="27.94" y="15.24" size="1.778" layer="27" rot="R90" display="off"/>
 </element>
-<element name="T1" library="triac" package="TO220BH" value="BT138-H" x="36.83" y="22.86"/>
-<element name="R1" library="rcl" package="R1206" value="380" x="2.54" y="-3.81"/>
-<element name="R2" library="rcl" package="R1206" value="330" x="2.54" y="-8.89"/>
-<element name="R3" library="rcl" package="R1206" value="39" x="2.54" y="-13.97"/>
-<element name="C1" library="rcl" package="C0805" value="0.01" x="2.54" y="-19.05"/>
-<element name="R4" library="rcl" package="R1206" value="330" x="2.54" y="-24.13"/>
-<element name="V220" library="con-amp-quick" package="02P" value="" x="-5.08" y="-20.32">
-<attribute name="OC_FARNELL" value="unknown" x="-5.08" y="-20.32" size="1.778" layer="27" display="off"/>
-<attribute name="OC_NEWARK" value="unknown" x="-5.08" y="-20.32" size="1.778" layer="27" display="off"/>
-<attribute name="MF" value="" x="-5.08" y="-20.32" size="1.778" layer="27" display="off"/>
-<attribute name="MPN" value="" x="-5.08" y="-20.32" size="1.778" layer="27" display="off"/>
+<element name="T1" library="triac" package="TO220BH" value="BT138-H" x="13.97" y="26.67"/>
+<element name="R1" library="rcl" package="R1206" value="380" x="22.86" y="8.89" rot="R180"/>
+<element name="R2" library="rcl" package="R1206" value="330" x="29.21" y="8.89" rot="R180"/>
+<element name="R3" library="rcl" package="R1206" value="39" x="22.86" y="6.35" rot="R180"/>
+<element name="C1" library="rcl" package="C0805" value="0.01" x="29.21" y="6.35"/>
+<element name="R4" library="rcl" package="R1206" value="330" x="39.37" y="12.7"/>
+<element name="V220" library="con-amp-quick" package="02P" value="" x="16.51" y="10.16">
+<attribute name="OC_FARNELL" value="unknown" x="16.51" y="10.16" size="1.778" layer="27" display="off"/>
+<attribute name="OC_NEWARK" value="unknown" x="16.51" y="10.16" size="1.778" layer="27" display="off"/>
+<attribute name="MF" value="" x="16.51" y="10.16" size="1.778" layer="27" display="off"/>
+<attribute name="MPN" value="" x="16.51" y="10.16" size="1.778" layer="27" display="off"/>
 </element>
-<element name="TEN" library="con-amp-quick" package="02P" value="" x="-12.7" y="-20.32">
-<attribute name="OC_FARNELL" value="unknown" x="-12.7" y="-20.32" size="1.778" layer="27" display="off"/>
-<attribute name="OC_NEWARK" value="unknown" x="-12.7" y="-20.32" size="1.778" layer="27" display="off"/>
-<attribute name="MF" value="" x="-12.7" y="-20.32" size="1.778" layer="27" display="off"/>
-<attribute name="MPN" value="" x="-12.7" y="-20.32" size="1.778" layer="27" display="off"/>
+<element name="TEN" library="con-amp-quick" package="02P" value="" x="8.89" y="10.16">
+<attribute name="OC_FARNELL" value="unknown" x="8.89" y="10.16" size="1.778" layer="27" display="off"/>
+<attribute name="OC_NEWARK" value="unknown" x="8.89" y="10.16" size="1.778" layer="27" display="off"/>
+<attribute name="MF" value="" x="8.89" y="10.16" size="1.778" layer="27" display="off"/>
+<attribute name="MPN" value="" x="8.89" y="10.16" size="1.778" layer="27" display="off"/>
 </element>
 </elements>
@@
 <contactref element="OK1" pad="6"/>
 <contactref element="R1" pad="1"/>
-<wire x1="1.118" y1="-3.81" x2="21.59" y2="25.4" width="0" layer="19" extent="1-1"/>
+<wire x1="24.13" y1="12.7" x2="24.13" y2="9.042" width="0.4064" layer="1"/>
+<wire x1="24.13" y1="9.042" x2="24.282" y2="8.89" width="0.4064" layer="1"/>
 </signal>
 <signal name="N$2">
@@
 <contactref element="R3" pad="2"/>
 <contactref element="V220" pad="1"/>
-<wire x1="3.962" y1="-3.81" x2="36.83" y2="16.51" width="0" layer="19" extent="1-1"/>
-<wire x1="3.962" y1="-13.97" x2="3.962" y2="-3.81" width="0" layer="19" extent="1-1"/>
-<wire x1="-6.35" y1="-20.32" x2="3.962" y2="-13.97" width="0" layer="19" extent="1-1"/>
+<wire x1="15.24" y1="10.16" x2="13.97" y2="11.43" width="0.4064" layer="1"/>
+<wire x1="13.97" y1="11.43" x2="13.97" y2="20.32" width="0.4064" layer="1"/>
+<wire x1="21.438" y1="8.89" x2="21.438" y2="11.582" width="0.4064" layer="1"/>
+<wire x1="21.438" y1="11.582" x2="20.32" y2="12.7" width="0.4064" layer="1"/>
+<wire x1="20.32" y1="12.7" x2="16.51" y2="12.7" width="0.4064" layer="1"/>
+<wire x1="16.51" y1="12.7" x2="15.24" y2="11.43" width="0.4064" layer="1"/>
+<wire x1="15.24" y1="11.43" x2="15.24" y2="10.16" width="0.4064" layer="1"/>
+<wire x1="21.438" y1="6.35" x2="21.438" y2="8.89" width="0.4064" layer="1"/>
 </signal>
 <signal name="N$3">
@@
 <contactref element="R2" pad="2"/>
 <contactref element="T1" pad="G"/>
-<wire x1="26.67" y1="25.4" x2="39.37" y2="16.51" width="0" layer="19" extent="1-1"/>
-<wire x1="3.962" y1="-8.89" x2="26.67" y2="25.4" width="0" layer="19" extent="1-1"/>
+<wire x1="24.13" y1="17.78" x2="17.78" y2="17.78" width="0.4064" layer="1"/>
+<wire x1="17.78" y1="17.78" x2="16.51" y2="19.05" width="0.4064" layer="1"/>
+<wire x1="16.51" y1="19.05" x2="16.51" y2="20.32" width="0.4064" layer="1"/>
+<wire x1="24.13" y1="17.78" x2="26.67" y2="17.78" width="0.4064" layer="1"/>
+<wire x1="26.67" y1="17.78" x2="27.94" y2="16.51" width="0.4064" layer="1"/>
+<wire x1="27.94" y1="16.51" x2="27.94" y2="9.042" width="0.4064" layer="1"/>
+<wire x1="27.94" y1="9.042" x2="27.788" y2="8.89" width="0.4064" layer="1"/>
 </signal>
 <signal name="N$4">
@@
 <contactref element="C1" pad="2"/>
 <contactref element="TEN" pad="2"/>
-<wire x1="1.118" y1="-8.89" x2="34.29" y2="16.51" width="0" layer="19" extent="1-1"/>
-<wire x1="3.49" y1="-19.05" x2="1.118" y2="-8.89" width="0" layer="19" extent="1-1"/>
-<wire x1="-11.43" y1="-20.32" x2="3.49" y2="-19.05" width="0" layer="19" extent="1-1"/>
+<wire x1="11.43" y1="20.32" x2="11.43" y2="11.43" width="0.4064" layer="1"/>
+<wire x1="11.43" y1="11.43" x2="10.16" y2="10.16" width="0.4064" layer="1"/>
+<wire x1="30.16" y1="6.35" x2="30.16" y2="8.418" width="0.4064" layer="1"/>
+<wire x1="30.16" y1="8.418" x2="30.632" y2="8.89" width="0.4064" layer="1"/>
+<wire x1="11.43" y1="20.32" x2="6.35" y2="20.32" width="0.4064" layer="1"/>
+<wire x1="6.35" y1="20.32" x2="5.08" y2="19.05" width="0.4064" layer="1"/>
+<wire x1="5.08" y1="19.05" x2="5.08" y2="6.35" width="0.4064" layer="1"/>
+<wire x1="5.08" y1="6.35" x2="7.62" y2="3.81" width="0.4064" layer="1"/>
+<wire x1="7.62" y1="3.81" x2="29.21" y2="3.81" width="0.4064" layer="1"/>
+<wire x1="29.21" y1="3.81" x2="30.48" y2="5.08" width="0.4064" layer="1"/>
+<wire x1="30.48" y1="5.08" x2="30.48" y2="6.03" width="0.4064" layer="1"/>
+<wire x1="30.48" y1="6.03" x2="30.16" y2="6.35" width="0.4064" layer="1"/>
 </signal>
 <signal name="N$6">
 <contactref element="R3" pad="1"/>
 <contactref element="C1" pad="1"/>
-<wire x1="1.118" y1="-13.97" x2="1.59" y2="-19.05" width="0" layer="19" extent="1-1"/>
+<wire x1="24.282" y1="6.35" x2="28.26" y2="6.35" width="0.4064" layer="1"/>
 </signal>
 <signal name="N$8">
 <contactref element="OK1" pad="1"/>
 <contactref element="R4" pad="2"/>
-<wire x1="3.962" y1="-24.13" x2="21.59" y2="17.78" width="0" layer="19" extent="1-1"/>
+<wire x1="31.75" y1="12.7" x2="40.792" y2="12.7" width="0" layer="19" extent="1-1"/>
 </signal>
 <signal name="N$9">
@@
 <contactref element="V220" pad="2"/>
 <contactref element="TEN" pad="1"/>
-<wire x1="-3.81" y1="-20.32" x2="-13.97" y2="-20.32" width="0" layer="19" extent="1-1"/>
+<wire x1="7.62" y1="10.16" x2="7.62" y2="8.89" width="0.4064" layer="1"/>
+<wire x1="7.62" y1="8.89" x2="8.89" y2="7.62" width="0.4064" layer="1"/>
+<wire x1="8.89" y1="7.62" x2="16.51" y2="7.62" width="0.4064" layer="1"/>
+<wire x1="16.51" y1="7.62" x2="17.78" y2="8.89" width="0.4064" layer="1"/>
+<wire x1="17.78" y1="8.89" x2="17.78" y2="10.16" width="0.4064" layer="1"/>
 </signal>
 </signals>

Commit message: ac dc
Parts:
- added C2: 0.01, rcl:C050-025X075
- added C3: 100uF 25V, rcl:E2,5-6
- added C4: 100n, rcl:C0805
- added C5, C6: 0.47 µF 250V, rcl:C150-072X183
- added D1, D2: 1N4007, diode:DO41-10
- added D3: 5.1V, diode:SMB
- added R5: 510, rcl:R0805
- added R6: 383, rcl:0207/7
- C1: value 0.01 -> 100uF 25V; device rcl:C0805 -> rcl:E2,5-6
- R1: value 380 -> 330; device rcl:R1206 -> rcl:0207/7
- R2: value 330 -> 39; device rcl:R1206 -> rcl:0207/7
- R3: value 39 -> 383; device rcl:R1206 -> rcl:0207/7
- moved C1 27.9 mm to (3.81, -5.08)
- moved R3 26.2 mm to (43.2, 22.9), turned to 0 degrees
- moved R1 25.5 mm to (48.3, 11.4), turned to 0 degrees
- moved R2 10.5 mm to (39.4, 6.35), turned to 0 degrees
Connections:
- new net +5V: C3.+, C4.1, D3.C, R5.2
- new net GND: C1.-, C3.-, C4.2, D2.A, D3.A
- new net N$11: C1.+, D1.C, R5.1
- new net N$13: R6.1
- new net N$14: C5.1, R6.2
- new net N$15: C5.2, C6.1
- new net N$5: C6.2, D1.A, D2.C
- net N$1: now also R3.1; no longer R1.1
- net N$2: now also R2.2; no longer R1.2
- net N$3: now also R1.2; no longer R2.2
- net N$4: now also C2.2, R1.1; no longer C1.2, R2.1
- net N$6: now also C2.1, R2.1; no longer C1.1, R3.1
Routing:
- net N$2: track 24.4 -> 19.1 mm
- net N$6: track 3.98 -> 0.00 mm
- net N$4: track 61.4 -> 58.2 mm
Changed lines of the file:
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@@
 <layer number="97" name="Info" color="7" fill="1" visible="no" active="no"/>
 <layer number="98" name="Guide" color="6" fill="1" visible="no" active="no"/>
+<layer number="99" name="SpiceOrder" color="5" fill="1" visible="no" active="no"/>
 </layers>
 <board>
@@
 </element>
 <element name="T1" library="triac" package="TO220BH" value="BT138-H" x="13.97" y="26.67"/>
-<element name="R1" library="rcl" package="R1206" value="380" x="22.86" y="8.89" rot="R180"/>
-<element name="R2" library="rcl" package="R1206" value="330" x="29.21" y="8.89" rot="R180"/>
-<element name="R3" library="rcl" package="R1206" value="39" x="22.86" y="6.35" rot="R180"/>
-<element name="C1" library="rcl" package="C0805" value="0.01" x="29.21" y="6.35"/>
 <element name="R4" library="rcl" package="R1206" value="330" x="39.37" y="12.7"/>
 <element name="V220" library="con-amp-quick" package="02P" value="" x="16.51" y="10.16">
@@
 <attribute name="MPN" value="" x="8.89" y="10.16" size="1.778" layer="27" display="off"/>
 </element>
+<element name="R3" library="rcl" package="0207/7" value="383" x="43.18" y="22.86"/>
+<element name="C2" library="rcl" package="C050-025X075" value="0.01" x="12.7" y="2.54"/>
+<element name="R1" library="rcl" package="0207/7" value="330" x="48.26" y="11.43"/>
+<element name="R2" library="rcl" package="0207/7" value="39" x="39.37" y="6.35"/>
+<element name="C1" library="rcl" package="E2,5-6" value="100uF 25V" x="3.81" y="-5.08"/>
+<element name="D1" library="diode" package="DO41-10" value="1N4007" x="6.35" y="-11.43"/>
+<element name="D2" library="diode" package="DO41-10" value="1N4007" x="6.35" y="-19.05"/>
+<element name="R5" library="rcl" package="R0805" value="510" x="2.54" y="-25.4"/>
+<element name="C3" library="rcl" package="E2,5-6" value="100uF 25V" x="3.81" y="-30.48"/>
+<element name="D3" library="diode" package="SMB" value="5.1V" x="3.81" y="-38.1"/>
+<element name="C4" library="rcl" package="C0805" value="100n" x="2.54" y="-43.18"/>
+<element name="R6" library="rcl" package="0207/7" value="383" x="5.08" y="-49.53"/>
+<element name="C5" library="rcl" package="C150-072X183" value="0.47 µF 250V" x="10.16" y="-57.15"/>
+<element name="C6" library="rcl" package="C150-072X183" value="0.47 µF 250V" x="10.16" y="-67.31"/>
 </elements>
 <signals>
 <signal name="N$1">
 <contactref element="OK1" pad="6"/>
-<contactref element="R1" pad="1"/>
 <wire x1="24.13" y1="12.7" x2="24.13" y2="9.042" width="0.4064" layer="1"/>
-<wire x1="24.13" y1="9.042" x2="24.282" y2="8.89" width="0.4064" layer="1"/>
+<contactref element="R3" pad="1"/>
+<wire x1="39.37" y1="22.86" x2="24.13" y2="9.042" width="0" layer="19" extent="1-1"/>
 </signal>
 <signal name="N$2">
 <contactref element="T1" pad="T2"/>
-<contactref element="R1" pad="2"/>
-<contactref element="R3" pad="2"/>
 <contactref element="V220" pad="1"/>
 <wire x1="15.24" y1="10.16" x2="13.97" y2="11.43" width="0.4064" layer="1"/>
 <wire x1="13.97" y1="11.43" x2="13.97" y2="20.32" width="0.4064" layer="1"/>
-<wire x1="21.438" y1="8.89" x2="21.438" y2="11.582" width="0.4064" layer="1"/>
 <wire x1="21.438" y1="11.582" x2="20.32" y2="12.7" width="0.4064" layer="1"/>
 <wire x1="20.32" y1="12.7" x2="16.51" y2="12.7" width="0.4064" layer="1"/>
 <wire x1="16.51" y1="12.7" x2="15.24" y2="11.43" width="0.4064" layer="1"/>
 <wire x1="15.24" y1="11.43" x2="15.24" y2="10.16" width="0.4064" layer="1"/>
-<wire x1="21.438" y1="6.35" x2="21.438" y2="8.89" width="0.4064" layer="1"/>
+<contactref element="R3" pad="2"/>
+<contactref element="R2" pad="2"/>
+<wire x1="21.438" y1="11.582" x2="46.99" y2="22.86" width="0" layer="19" extent="1-1"/>
+<wire x1="43.18" y1="6.35" x2="15.24" y2="10.16" width="0" layer="19" extent="1-1"/>
 </signal>
 <signal name="N$3">
 <contactref element="OK1" pad="4"/>
-<contactref element="R2" pad="2"/>
 <contactref element="T1" pad="G"/>
 <wire x1="24.13" y1="17.78" x2="17.78" y2="17.78" width="0.4064" layer="1"/>
@@
 <wire x1="26.67" y1="17.78" x2="27.94" y2="16.51" width="0.4064" layer="1"/>
 <wire x1="27.94" y1="16.51" x2="27.94" y2="9.042" width="0.4064" layer="1"/>
-<wire x1="27.94" y1="9.042" x2="27.788" y2="8.89" width="0.4064" layer="1"/>
+<contactref element="R1" pad="2"/>
+<wire x1="52.07" y1="11.43" x2="27.94" y2="9.042" width="0" layer="19" extent="1-1"/>
 </signal>
 <signal name="N$4">
-<contactref element="R2" pad="1"/>
 <contactref element="T1" pad="T1"/>
-<contactref element="C1" pad="2"/>
 <contactref element="TEN" pad="2"/>
 <wire x1="11.43" y1="20.32" x2="11.43" y2="11.43" width="0.4064" layer="1"/>
 <wire x1="11.43" y1="11.43" x2="10.16" y2="10.16" width="0.4064" layer="1"/>
-<wire x1="30.16" y1="6.35" x2="30.16" y2="8.418" width="0.4064" layer="1"/>
-<wire x1="30.16" y1="8.418" x2="30.632" y2="8.89" width="0.4064" layer="1"/>
 <wire x1="11.43" y1="20.32" x2="6.35" y2="20.32" width="0.4064" layer="1"/>
 <wire x1="6.35" y1="20.32" x2="5.08" y2="19.05" width="0.4064" layer="1"/>
@@
 <wire x1="29.21" y1="3.81" x2="30.48" y2="5.08" width="0.4064" layer="1"/>
 <wire x1="30.48" y1="5.08" x2="30.48" y2="6.03" width="0.4064" layer="1"/>
-<wire x1="30.48" y1="6.03" x2="30.16" y2="6.35" width="0.4064" layer="1"/>
-</signal>
-<signal name="N$6">
-<contactref element="R3" pad="1"/>
-<contactref element="C1" pad="1"/>
-<wire x1="24.282" y1="6.35" x2="28.26" y2="6.35" width="0.4064" layer="1"/>
+<contactref element="C2" pad="2"/>
+<contactref element="R1" pad="1"/>
+<wire x1="15.24" y1="2.54" x2="7.62" y2="3.81" width="0" layer="19" extent="1-1"/>
+<wire x1="44.45" y1="11.43" x2="15.24" y2="2.54" width="0" layer="19" extent="1-1"/>
 </signal>
 <signal name="N$8">
@@
 <wire x1="17.78" y1="8.89" x2="17.78" y2="10.16" width="0.4064" layer="1"/>
 </signal>
+<signal name="N$6">
+<contactref element="C2" pad="1"/>
+<contactref element="R2" pad="1"/>
+<wire x1="10.16" y1="2.54" x2="35.56" y2="6.35" width="0" layer="19" extent="1-1"/>
+</signal>
+<signal name="N$5">
+<contactref element="D2" pad="C"/>
+<contactref element="D1" pad="A"/>
+<contactref element="C6" pad="2"/>
+<wire x1="1.27" y1="-19.05" x2="17.653" y2="-67.31" width="0" layer="19" extent="1-1"/>
+<wire x1="11.43" y1="-11.43" x2="1.27" y2="-19.05" width="0" layer="19" extent="1-1"/>
+</signal>
+<signal name="N$11">
+<contactref element="D1" pad="C"/>
+<contactref element="C1" pad="+"/>
+<contactref element="R5" pad="1"/>
+<wire x1="1.27" y1="-11.43" x2="1.59" y2="-25.4" width="0" layer="19" extent="1-1"/>
+<wire x1="2.54" y1="-5.08" x2="1.27" y2="-11.43" width="0" layer="19" extent="1-1"/>
+</signal>
+<signal name="+5V">
+<contactref element="D3" pad="C"/>
+<contactref element="C4" pad="1"/>
+<contactref element="C3" pad="+"/>
+<contactref element="R5" pad="2"/>
+<wire x1="1.61" y1="-38.1" x2="1.59" y2="-43.18" width="0" layer="19" extent="1-1"/>
+<wire x1="2.54" y1="-30.48" x2="1.61" y2="-38.1" width="0" layer="19" extent="1-1"/>
+<wire x1="3.49" y1="-25.4" x2="2.54" y2="-30.48" width="0" layer="19" extent="1-1"/>
+</signal>
+<signal name="GND">
+<contactref element="D2" pad="A"/>
+<contactref element="D3" pad="A"/>
+<contactref element="C1" pad="-"/>
+<contactref element="C4" pad="2"/>
+<contactref element="C3" pad="-"/>
+<wire x1="6.01" y1="-38.1" x2="3.49" y2="-43.18" width="0" layer="19" extent="1-1"/>
+<wire x1="5.08" y1="-30.48" x2="6.01" y2="-38.1" width="0" layer="19" extent="1-1"/>
+<wire x1="11.43" y1="-19.05" x2="5.08" y2="-30.48" width="0" layer="19" extent="1-1"/>
+<wire x1="5.08" y1="-5.08" x2="11.43" y2="-19.05" width="0" layer="19" extent="1-1"/>
+</signal>
+<signal name="N$13">
+<contactref element="R6" pad="1"/>
+</signal>
+<signal name="N$14">
+<contactref element="C5" pad="1"/>
+<contactref element="R6" pad="2"/>
+<wire x1="8.89" y1="-49.53" x2="2.667" y2="-57.15" width="0" layer="19" extent="1-1"/>
+</signal>
+<signal name="N$15">
+<contactref element="C5" pad="2"/>
+<contactref element="C6" pad="1"/>
+<wire x1="17.653" y1="-57.15" x2="2.667" y2="-67.31" width="0" layer="19" extent="1-1"/>
+</signal>
 </signals>

Commit message: layout changes
Parts:
- added C7: 1uF, rcl:C0805
- added C8: 100n, rcl:C0805
- added IC1: STM8S003F3, stm8:TSSOP20
- added SV1: (no value), con-lstb:MA04-1
- added U$1: MCP1825SOT-223-3, SteelCaveRobotics-Power:SOT-223
- D1, D2: value 1N4007 -> Semikron S1Y; device diode:DO41-10 -> diode:SMA
- moved C6 94.4 mm to (19.1, 26.7), turned to 270 degrees
- moved C5 83.8 mm to (11.4, 26.7), turned to 90 degrees
- moved C4 68.3 mm to (14.0, 24.1), turned to 270 degrees
- moved R6 65.6 mm to (15.2, 15.2), turned to 180 degrees
- moved D3 62.6 mm to (10.2, 24.1), turned to 270 degrees
- moved R5 59.5 mm to (19.1, 31.8)
- moved C3 54.6 mm to (5.08, 24.1), turned to 270 degrees
- moved D2 48.7 mm to (19.1, 27.9)
- moved D1 36.6 mm to (19.1, 22.9), turned to 180 degrees
- moved C1 35.6 mm to (5.08, 30.5), turned to 270 degrees
- moved T1 27.3 mm to (38.1, 14.0)
- moved R4 22.2 mm to (30.5, 33.0), turned to 270 degrees
- moved R3 21.0 mm to (24.1, 14.0), turned to 180 degrees
- moved R2 18.3 mm to (24.1, 16.5), turned to 180 degrees
- moved R1 17.8 mm to (30.5, 10.2), turned to 90 degrees
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Connections:
- removed net +5V: C3.+, C4.1, D3.C, R5.2
- removed net GND: C1.-, C3.-, C4.2, D2.A, D3.A
- removed net N$13: R6.1
- new net +3V3: IC1.9, R4.1, SV1.1, U$1.3
- new net L: R2.2, R3.2, R6.1, T1.T2, V220.1
- new net N: C1.-, C3.-, C4.2, C7.2, C8.2, D1.A, D3.A, IC1.7, SV1.3, TEN.1, U$1.2, V220.2
- new net N$12: C3.+, C4.1, D3.C, R5.2, U$1.1
- net N$10: now also IC1.19
- net N$11: now also D2.C; no longer D1.C
- net N$2: now also C7.1, IC1.8; no longer R2.2, R3.2, T1.T2, V220.1
- net N$5: now also D1.C, D2.A; no longer D1.A, D2.C
- net N$7: now also C8.1, IC1.4, SV1.4; no longer TEN.1, V220.2
- net N$9: now also IC1.18, SV1.2; no longer R4.1
Routing:
- net N: track 0.00 -> 87.4 mm
- net N$12: track 0.00 -> 44.2 mm
- net N$4: track 58.2 -> 15.8 mm
- net L: track 0.00 -> 37.4 mm
- net N$10: track 0.00 -> 22.0 mm
- net N$8: track 0.00 -> 18.6 mm
- net N$11: track 0.00 -> 17.3 mm
- net N$2: track 19.1 -> 4.70 mm
- net N$7: track 13.8 -> 0.00 mm
- net N$5: track 0.00 -> 9.59 mm
- net N$3: track 21.2 -> 29.6 mm
- net N$15: track 0.00 -> 7.62 mm
- net N$6: track 0.00 -> 7.40 mm
- net N$1: track 3.66 -> 11.0 mm
- net N$14: track 0.00 -> 3.94 mm

Commit message: last version of laminator
Parts:
- moved R3 19.1 mm to (5.08, 12.7), turned to 270 degrees
- moved T1 16.6 mm to (24.1, 5.08), turned to 270 degrees
- moved R1 15.5 mm to (15.2, 12.7)
- moved C2 14.5 mm to (12.7, 12.7)
- moved R2 14.5 mm to (10.2, 12.7), turned to 270 degrees
- moved R4 11.5 mm to (29.2, 21.6)
- moved V220 10.2 mm to (6.35, 5.08)
- moved TEN 10.2 mm to (12.7, 5.08)
- moved OK1 8.78 mm to (27.3, 14.3)
- moved R6 8.03 mm to (7.62, 12.7), turned to 90 degrees
Routing:
- net N$10: track 22.0 -> 3.57 mm
- net N: track 87.4 -> 71.9 mm
- net N$1: track 11.0 -> 21.3 mm
- net N$8: track 18.6 -> 9.77 mm
- net L: track 37.4 -> 31.1 mm
- net N$2: track 4.70 -> 0.00 mm
- net N$4: track 15.8 -> 11.2 mm
- net N$6: track 7.40 -> 3.07 mm
- net N$3: track 29.6 -> 32.3 mm
- net N$14: track 3.94 -> 5.66 mm
