File: laminator.sch (EAGLE design)
At the start: 9 parts, among them T1 BT138-H

Commit message: ac dc
Parts:
- added C2: 0.01, rcl:C-EU050-025X075
- added C3: 100uF 25V, rcl:CPOL-EUE2.5-6
- added C4: 100n, rcl:C-EUC0805
- added C5, C6: 0.47 µF 250V, rcl:C-EU150-072X183
- added D1, D2: 1N4007, diode:1N4004
- added D3: 5.1V, diode:ZENER-DIODESMB
- added R5: 510, rcl:R-EU_R0805
- added R6: 383, rcl:R-EU_0207/7
- C1: value 0.01 -> 100uF 25V; device rcl:C-EUC0805 -> rcl:CPOL-EUE2.5-6
- R1: value 380 -> 330; device rcl:R-EU_R1206 -> rcl:R-EU_0207/7
- R2: value 330 -> 39; device rcl:R-EU_R1206 -> rcl:R-EU_0207/7
- R3: value 39 -> 383; device rcl:R-EU_R1206 -> rcl:R-EU_0207/7
Connections:
- new net +5V: C3.+, C4.1, D3.C, R5.2
- new net GND: C1.-, C3.-, C4.2, D2.A, D3.A
- new net N$11: C1.+, D1.C, R5.1
- new net N$13: R6.1
- new net N$14: C5.1, R6.2
- new net N$15: C5.2, C6.1
- new net N$5: C6.2, D1.A, D2.C
- net N$1: now also R3.1; no longer R1.1
- net N$2: now also R2.2; no longer R1.2
- net N$3: now also R1.2; no longer R2.2
- net N$4: now also C2.2, R1.1; no longer C1.2, R2.1
- net N$6: now also C2.1, R2.1; no longer C1.1, R3.1
Other:
- moved on the sheet: R1, R2, R3
Changed lines of the file:
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@@
 <layer number="97" name="Info" color="7" fill="1" visible="yes" active="yes"/>
 <layer number="98" name="Guide" color="6" fill="1" visible="yes" active="yes"/>
+<layer number="99" name="SpiceOrder" color="5" fill="1" visible="yes" active="yes"/>
 </layers>
 <schematic xreflabel="%F%N/%S.%C%R" xrefpart="/%S.%C%R">
@@
 <part name="OK1" library="optocoupler" deviceset="MOC30*" device="" technology="41M"/>
 <part name="T1" library="triac" deviceset="BT138" device="-H"/>
-<part name="R1" library="rcl" deviceset="R-EU_" device="R1206" value="380"/>
-<part name="R2" library="rcl" deviceset="R-EU_" device="R1206" value="330"/>
-<part name="R3" library="rcl" deviceset="R-EU_" device="R1206" value="39"/>
-<part name="C1" library="rcl" deviceset="C-EU" device="C0805" value="0.01"/>
 <part name="R4" library="rcl" deviceset="R-EU_" device="R1206" value="330"/>
 <part name="V220" library="con-amp-quick" deviceset="M02" device=""/>
 <part name="TEN" library="con-amp-quick" deviceset="M02" device=""/>
+<part name="R3" library="rcl" deviceset="R-EU_" device="0207/7" value="383"/>
+<part name="C2" library="rcl" deviceset="C-EU" device="050-025X075" value="0.01"/>
+<part name="R1" library="rcl" deviceset="R-EU_" device="0207/7" value="330"/>
+<part name="R2" library="rcl" deviceset="R-EU_" device="0207/7" value="39"/>
+<part name="C1" library="rcl" deviceset="CPOL-EU" device="E2.5-6" value="100uF 25V"/>
+<part name="D1" library="diode" deviceset="1N4004" device="" value="1N4007"/>
+<part name="D2" library="diode" deviceset="1N4004" device="" value="1N4007"/>
+<part name="R5" library="rcl" deviceset="R-EU_" device="R0805" value="510"/>
+<part name="C3" library="rcl" deviceset="CPOL-EU" device="E2.5-6" value="100uF 25V"/>
+<part name="D3" library="diode" deviceset="ZENER-DIODE" device="SMB" value="5.1V"/>
+<part name="C4" library="rcl" deviceset="C-EU" device="C0805" value="100n"/>
+<part name="GND1" library="supply1" deviceset="GND" device=""/>
+<part name="P+1" library="supply1" deviceset="+5V" device=""/>
+<part name="R6" library="rcl" deviceset="R-EU_" device="0207/7" value="383"/>
+<part name="C5" library="rcl" deviceset="C-EU" device="150-072X183" value="0.47 µF 250V"/>
+<part name="C6" library="rcl" deviceset="C-EU" device="150-072X183" value="0.47 µF 250V"/>
 </parts>
 <sheets>
@@
 <instance part="OK1" gate="-1" x="10.16" y="10.16"/>
 <instance part="T1" gate="G$1" x="38.1" y="7.62"/>
-<instance part="R1" gate="G$1" x="27.94" y="15.24"/>
-<instance part="R2" gate="G$1" x="27.94" y="-2.54" rot="R90"/>
-<instance part="R3" gate="G$1" x="45.72" y="5.08" rot="R90"/>
-<instance part="C1" gate="G$1" x="45.72" y="-5.08"/>
 <instance part="R4" gate="G$1" x="-10.16" y="15.24"/>
 <instance part="V220" gate="G$1" x="76.2" y="10.16" rot="R180"/>
 <instance part="TEN" gate="G$1" x="76.2" y="-2.54" rot="R180"/>
+<instance part="R3" gate="G$1" x="27.94" y="15.24"/>
+<instance part="C2" gate="G$1" x="45.72" y="-5.08"/>
+<instance part="R1" gate="G$1" x="27.94" y="-2.54" rot="R90"/>
+<instance part="R2" gate="G$1" x="45.72" y="5.08" rot="R90"/>
+<instance part="C1" gate="G$1" x="55.88" y="45.72"/>
+<instance part="D1" gate="1" x="43.18" y="50.8"/>
+<instance part="D2" gate="1" x="35.56" y="43.18" rot="R90"/>
+<instance part="R5" gate="G$1" x="68.58" y="50.8"/>
+<instance part="C3" gate="G$1" x="86.36" y="45.72"/>
+<instance part="D3" gate="G$1" x="78.74" y="45.72" rot="R90"/>
+<instance part="C4" gate="G$1" x="101.6" y="45.72"/>
+<instance part="GND1" gate="1" x="116.84" y="30.48"/>
+<instance part="P+1" gate="1" x="116.84" y="55.88"/>
+<instance part="R6" gate="G$1" x="7.62" y="50.8"/>
+<instance part="C5" gate="G$1" x="17.78" y="50.8" rot="R90"/>
+<instance part="C6" gate="G$1" x="27.94" y="50.8" rot="R90"/>
 </instances>
 <busses>
@@
 <segment>
 <pinref part="OK1" gate="-1" pin="A2"/>
-<pinref part="R1" gate="G$1" pin="1"/>
 <wire x1="20.32" y1="15.24" x2="22.86" y2="15.24" width="0.1524" layer="91"/>
+<pinref part="R3" gate="G$1" pin="1"/>
 </segment>
 </net>
@@
 <pinref part="T1" gate="G$1" pin="A2"/>
 <wire x1="38.1" y1="12.7" x2="38.1" y2="15.24" width="0.1524" layer="91"/>
-<pinref part="R1" gate="G$1" pin="2"/>
 <wire x1="38.1" y1="15.24" x2="33.02" y2="15.24" width="0.1524" layer="91"/>
-<pinref part="R3" gate="G$1" pin="2"/>
 <wire x1="45.72" y1="10.16" x2="45.72" y2="15.24" width="0.1524" layer="91"/>
 <wire x1="45.72" y1="15.24" x2="38.1" y2="15.24" width="0.1524" layer="91"/>
@@
 <wire x1="68.58" y1="10.16" x2="63.5" y2="10.16" width="0.1524" layer="91"/>
 <wire x1="63.5" y1="10.16" x2="63.5" y2="15.24" width="0.1524" layer="91"/>
+<pinref part="R3" gate="G$1" pin="2"/>
+<pinref part="R2" gate="G$1" pin="2"/>
 </segment>
 </net>
@@
 <segment>
 <pinref part="OK1" gate="-1" pin="A1"/>
-<pinref part="R2" gate="G$1" pin="2"/>
 <wire x1="20.32" y1="5.08" x2="27.94" y2="5.08" width="0.1524" layer="91"/>
 <wire x1="27.94" y1="5.08" x2="27.94" y2="2.54" width="0.1524" layer="91"/>
@@
 <wire x1="27.94" y1="7.62" x2="27.94" y2="5.08" width="0.1524" layer="91"/>
 <junction x="27.94" y="5.08"/>
+<pinref part="R1" gate="G$1" pin="2"/>
 </segment>
 </net>
 <net name="N$4" class="0">
 <segment>
-<pinref part="R2" gate="G$1" pin="1"/>
 <wire x1="27.94" y1="-7.62" x2="27.94" y2="-12.7" width="0.1524" layer="91"/>
 <pinref part="T1" gate="G$1" pin="A1"/>
 <wire x1="27.94" y1="-12.7" x2="38.1" y2="-12.7" width="0.1524" layer="91"/>
 <wire x1="38.1" y1="-12.7" x2="38.1" y2="5.08" width="0.1524" layer="91"/>
-<pinref part="C1" gate="G$1" pin="2"/>
 <wire x1="45.72" y1="-10.16" x2="45.72" y2="-12.7" width="0.1524" layer="91"/>
 <wire x1="45.72" y1="-12.7" x2="38.1" y2="-12.7" width="0.1524" layer="91"/>
@@
 <pinref part="TEN" gate="G$1" pin="2"/>
 <wire x1="63.5" y1="-5.08" x2="68.58" y2="-5.08" width="0.1524" layer="91"/>
+<pinref part="C2" gate="G$1" pin="2"/>
+<pinref part="R1" gate="G$1" pin="1"/>
 </segment>
 </net>
 <net name="N$6" class="0">
 <segment>
-<pinref part="R3" gate="G$1" pin="1"/>
-<pinref part="C1" gate="G$1" pin="1"/>
 <wire x1="45.72" y1="0" x2="45.72" y2="-2.54" width="0.1524" layer="91"/>
+<pinref part="C2" gate="G$1" pin="1"/>
+<pinref part="R2" gate="G$1" pin="1"/>
 </segment>
 </net>
@@
 </segment>
 </net>
+<net name="N$5" class="0">
+<segment>
+<pinref part="D2" gate="1" pin="C"/>
+<wire x1="35.56" y1="45.72" x2="35.56" y2="50.8" width="0.1524" layer="91"/>
+<pinref part="D1" gate="1" pin="A"/>
+<wire x1="35.56" y1="50.8" x2="40.64" y2="50.8" width="0.1524" layer="91"/>
+<pinref part="C6" gate="G$1" pin="2"/>
+<wire x1="33.02" y1="50.8" x2="35.56" y2="50.8" width="0.1524" layer="91"/>
+<junction x="35.56" y="50.8"/>
+</segment>
+</net>
+<net name="N$11" class="0">
+<segment>
+<pinref part="D1" gate="1" pin="C"/>
+<pinref part="C1" gate="G$1" pin="+"/>
+<wire x1="45.72" y1="50.8" x2="55.88" y2="50.8" width="0.1524" layer="91"/>
+<wire x1="55.88" y1="50.8" x2="55.88" y2="48.26" width="0.1524" layer="91"/>
+<pinref part="R5" gate="G$1" pin="1"/>
+<wire x1="55.88" y1="50.8" x2="63.5" y2="50.8" width="0.1524" layer="91"/>
+<junction x="55.88" y="50.8"/>
+</segment>
+</net>
+<net name="+5V" class="0">
+<segment>
+<pinref part="R5" gate="G$1" pin="2"/>
+<pinref part="D3" gate="G$1" pin="C"/>
+<wire x1="73.66" y1="50.8" x2="78.74" y2="50.8" width="0.1524" layer="91"/>
+<wire x1="78.74" y1="50.8" x2="78.74" y2="48.26" width="0.1524" layer="91"/>
+<pinref part="C3" gate="G$1" pin="+"/>
+<wire x1="78.74" y1="50.8" x2="86.36" y2="50.8" width="0.1524" layer="91"/>
+<wire x1="86.36" y1="50.8" x2="86.36" y2="48.26" width="0.1524" layer="91"/>
+<junction x="78.74" y="50.8"/>
+<pinref part="C4" gate="G$1" pin="1"/>
+<wire x1="86.36" y1="50.8" x2="101.6" y2="50.8" width="0.1524" layer="91"/>
+<wire x1="101.6" y1="50.8" x2="101.6" y2="48.26" width="0.1524" layer="91"/>
+<junction x="86.36" y="50.8"/>
+<pinref part="P+1" gate="1" pin="+5V"/>
+<wire x1="101.6" y1="50.8" x2="116.84" y2="50.8" width="0.1524" layer="91"/>
+<wire x1="116.84" y1="50.8" x2="116.84" y2="53.34" width="0.1524" layer="91"/>
+<junction x="101.6" y="50.8"/>
+</segment>
+</net>
+<net name="GND" class="0">
+<segment>
+<pinref part="D2" gate="1" pin="A"/>
+<wire x1="35.56" y1="40.64" x2="35.56" y2="35.56" width="0.1524" layer="91"/>
+<pinref part="C1" gate="G$1" pin="-"/>
+<wire x1="35.56" y1="35.56" x2="55.88" y2="35.56" width="0.1524" layer="91"/>
+<wire x1="55.88" y1="35.56" x2="55.88" y2="40.64" width="0.1524" layer="91"/>
+<pinref part="D3" gate="G$1" pin="A"/>
+<wire x1="55.88" y1="35.56" x2="78.74" y2="35.56" width="0.1524" layer="91"/>
+<wire x1="78.74" y1="35.56" x2="78.74" y2="43.18" width="0.1524" layer="91"/>
+<junction x="55.88" y="35.56"/>
+<pinref part="C3" gate="G$1" pin="-"/>
+<wire x1="78.74" y1="35.56" x2="86.36" y2="35.56" width="0.1524" layer="91"/>
+<wire x1="86.36" y1="35.56" x2="86.36" y2="40.64" width="0.1524" layer="91"/>
+<junction x="78.74" y="35.56"/>
+<pinref part="C4" gate="G$1" pin="2"/>
+<wire x1="86.36" y1="35.56" x2="101.6" y2="35.56" width="0.1524" layer="91"/>
+<wire x1="101.6" y1="35.56" x2="101.6" y2="40.64" width="0.1524" layer="91"/>
+<junction x="86.36" y="35.56"/>
+<pinref part="GND1" gate="1" pin="GND"/>
+<wire x1="101.6" y1="35.56" x2="116.84" y2="35.56" width="0.1524" layer="91"/>
+<wire x1="116.84" y1="35.56" x2="116.84" y2="33.02" width="0.1524" layer="91"/>
+<junction x="101.6" y="35.56"/>
+</segment>
+</net>
+<net name="N$13" class="0">
+<segment>
+<pinref part="R6" gate="G$1" pin="1"/>
+<wire x1="0" y1="50.8" x2="2.54" y2="50.8" width="0.1524" layer="91"/>
+</segment>
+</net>
+<net name="N$14" class="0">
+<segment>
+<pinref part="C5" gate="G$1" pin="1"/>
+<pinref part="R6" gate="G$1" pin="2"/>
+<wire x1="15.24" y1="50.8" x2="12.7" y2="50.8" width="0.1524" layer="91"/>
+</segment>
+</net>
+<net name="N$15" class="0">
+<segment>
+<pinref part="C5" gate="G$1" pin="2"/>
+<pinref part="C6" gate="G$1" pin="1"/>
+<wire x1="22.86" y1="50.8" x2="25.4" y2="50.8" width="0.1524" layer="91"/>
+</segment>
+</net>

Commit message: layout changes
Parts:
- added C7: 1uF, rcl:C-EUC0805
- added C8: 100n, rcl:C-EUC0805
- added IC1: STM8S003F3, stm8:STM8S003F3
- added SV1: (no value), con-lstb:MA04-1
- added U$1: MCP1825SOT-223-3, SteelCaveRobotics-Power:MCP1825SOT-223-3
- D1, D2: value 1N4007 -> Semikron S1Y; device diode:1N4004 -> diode:MBRA340T3
Connections:
- removed net +5V: C3.+, C4.1, D3.C, R5.2
- removed net GND: C1.-, C3.-, C4.2, D2.A, D3.A
- removed net N$13: R6.1
- new net +3V3: IC1.VDD, R4.1, SV1.1, U$1.+3V3
- new net L: R2.2, R3.2, R6.1, T1.A2, V220.1
- new net N: C1.-, C3.-, C4.2, C7.2, C8.2, D1.A, D3.A, IC1.GND, SV1.3, TEN.1, U$1.GND@2, V220.2
- new net N$12: C3.+, C4.1, D3.C, R5.2, U$1.IN
- net N$10: now also IC1.PD2/AIN3/[TIM2_CH3]
- net N$11: now also D2.C; no longer D1.C
- net N$2: now also C7.1, IC1.VCAP; no longer R2.2, R3.2, T1.A2, V220.1
- net N$5: now also D1.C, D2.A; no longer D1.A, D2.C
- net N$7: now also C8.1, IC1.!RST, SV1.4; no longer TEN.1, V220.2
- net N$9: now also IC1.PD1/SWIM, SV1.2; no longer R4.1
Other:
- moved on the sheet: C1, C2, C3, C4, C5, C6, D3, OK1, R1, R2, R3, R4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

Commit message: last version of laminator
Other:
- moved on the sheet: V220
Changed lines of the file:
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@@
 <?xml version="1.0" encoding="utf-8"?>
 <!DOCTYPE eagle SYSTEM "eagle.dtd">
-<eagle version="7.4.0">
+<eagle version="7.3.0">
 <drawing>
 <settings>
@@
 <instance part="T1" gate="G$1" x="-127" y="-25.4" rot="R180"/>
 <instance part="R4" gate="G$1" x="-78.74" y="-33.02" rot="R180"/>
-<instance part="V220" gate="G$1" x="114.3" y="10.16" rot="R180"/>
+<instance part="V220" gate="G$1" x="-190.5" y="5.08" rot="R180"/>
 <instance part="TEN" gate="G$1" x="-165.1" y="-15.24"/>
 <instance part="R3" gate="G$1" x="-116.84" y="-33.02" rot="R180"/>
@@
 <segment>
 <pinref part="V220" gate="G$1" pin="1"/>
-<wire x1="106.68" y1="10.16" x2="101.6" y2="10.16" width="0.1524" layer="91"/>
-<label x="101.6" y="10.16" size="1.778" layer="95"/>
+<wire x1="-198.12" y1="5.08" x2="-203.2" y2="5.08" width="0.1524" layer="91"/>
+<label x="-203.2" y="5.08" size="1.778" layer="95"/>
 </segment>
 <segment>
@@
 <segment>
 <pinref part="V220" gate="G$1" pin="2"/>
-<wire x1="106.68" y1="7.62" x2="101.6" y2="7.62" width="0.1524" layer="91"/>
-<label x="101.6" y="7.62" size="1.778" layer="95"/>
-</segment>
-<segment>
+<wire x1="-198.12" y1="2.54" x2="-203.2" y2="2.54" width="0.1524" layer="91"/>
+<label x="-203.2" y="2.54" size="1.778" layer="95"/>
+</segment>
+<segment>
